Commit message: Changed torso_ur3 position

File: rb1_base_description/robots/rb1_dual_ur3.urdf.xacro (robot description, xacro)
@@ -79,5 +79,5 @@
 	<!-- TORSO & ARMS -->
 	<xacro:torso_ur3 prefix="$(arg prefix)" parent="$(arg prefix)base_link">
-		<origin xyz="-0.1 0.0 0.1718" rpy="0.0 0.0 0.0"/>
+		<origin xyz="0.0 0.0 0.19" rpy="0.0 0.0 0.0"/>
 	</xacro:torso_ur3>
 	<xacro:arg name="transmission_hw_interface" default="hardware_interface/PositionJointInterface"/>
